Commit message: change hardcoded paths to relative

File: src/sucky/urdf/robot_core.xacro (robot description, xacro)
@@ -47,5 +47,5 @@
       <origin xyz="0 0 0" rpy="0 0 ${pi/2}"/>
       <geometry>
-        <mesh filename="file://$(find sucky)/meshes/Sucky.stl" scale="1 1 1" />
+        <mesh filename="package://sucky/meshes/Sucky.stl" scale="1 1 1" />
       </geometry>
       <material name="orange"/>
@@ -54,5 +54,5 @@
       <origin xyz="0 0 0" rpy="0 0 ${pi/2}"/>
       <geometry>
-        <mesh filename="file://$(find sucky)/meshes/Sucky.stl" scale="1 1 1" />
+        <mesh filename="package://sucky/meshes/Sucky.stl" scale="1 1 1" />
       </geometry>
     </collision>
@@ -68,5 +68,5 @@
       <visual>
           <geometry>
-              <mesh filename="file://$(find sucky)/meshes/Big_Wheel.stl" scale="0.001 0.001 0.001" />
+              <mesh filename="package://sucky/meshes/Big_Wheel.stl" scale="0.001 0.001 0.001" />
           </geometry>
           <material name="black"/>
@@ -74,5 +74,5 @@
       <collision>
           <geometry>
-              <mesh filename="file://$(find sucky)/meshes/Big_Wheel.stl" scale="0.001 0.001 0.001" />
+              <mesh filename="package://sucky/meshes/Big_Wheel.stl" scale="0.001 0.001 0.001" />
           </geometry>
       </collision>
@@ -88,5 +88,5 @@
       <visual>
           <geometry>
-              <mesh filename="file://$(find sucky)/meshes/Big_Wheel.stl" scale="0.001 0.001 0.001" />
+              <mesh filename="package://sucky/meshes/Big_Wheel.stl" scale="0.001 0.001 0.001" />
           </geometry>
           <material name="black"/>
@@ -94,5 +94,5 @@
       <collision>
           <geometry>
-              <mesh filename="file://$(find sucky)/meshes/Big_Wheel.stl" scale="0.001 0.001 0.001" />
+              <mesh filename="package://sucky/meshes/Big_Wheel.stl" scale="0.001 0.001 0.001" />
           </geometry>
       </collision>

File: src/sucky/urdf/sensor_d455.urdf.xacro (robot description, xacro)
@@ -68,5 +68,5 @@
         <geometry>
           <!-- <box size="${d455_cam_depth} ${d455_cam_width} ${d455_cam_height}"/> -->
-	        <mesh filename="file://$(find sucky)/meshes/d455.stl" scale="0.001 0.001 0.001" />
+	        <mesh filename="package://sucky/meshes/d455.stl" scale="0.001 0.001 0.001" />
         </geometry>
         <material name="aluminum"/>

File: src/sucky/urdf/sensor_d455_usb_plug.urdf.xacro (robot description, xacro)
@@ -33,5 +33,5 @@
         <geometry>
           <!--box size="0.044850 0.008 0.0185" /-->
-          <mesh filename="file://$(find sucky)/meshes/d455_plug.stl" />
+          <mesh filename="package://sucky/meshes/d455_plug.stl" />
         </geometry>
         <material name="plastic"/>
@@ -41,5 +41,5 @@
         <geometry>
           <!--box size="0.044850 0.008 0.0185" /-->
-          <mesh filename="file://$(find sucky)/meshes/d455_plug_collision.stl" />
+          <mesh filename="package://sucky/meshes/d455_plug_collision.stl" />
         </geometry>
       </collision>

File: src/sucky/urdf/sensor_sick.xacro (robot description, xacro)
@@ -8,5 +8,5 @@
             <origin xyz="0 0 0" rpy="0 0 0"/>
             <geometry>
-                <mesh filename="file://$(find sucky)/meshes/sick781.stl" />
+                <mesh filename="package://sucky/meshes/sick781.stl" />
             </geometry>
             <material name="grey"/>
